File: winter2026/ecen476/motors/gazelem_main_motors_pcb_design/gazelem_main_motors_pcb_design.kicad_pcb (KiCad board)
At the start: 2 copper layers, 43 x 67 mm, 9 parts, among them J1 Conn_01x04_Pin, J2 Conn_01x04_Pin

Commit message: Completed 555 hw 5
Routing:
- added copper zone on B.Cu, net DIR- 1
- removed copper zone on F.Cu, net DIR- 1
Changed lines of the file:
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@@
 		(tenting front back)
 		(pcbplotparams
-			(layerselection 0x00000000_00000000_55555555_5755f57b)
+			(layerselection 0x00000000_00000000_55555555_5755f5ff)
 			(plot_on_all_layers_selection 0x00000000_00000000_00000000_00000000)
 			(disableapertmacros no)
@@
 			(drillshape 0)
 			(scaleselection 1)
-			(outputdirectory "fabrication_outputs/")
+			(outputdirectory "fabrication_outputs_march5_redo/")
 		)
 	)
@@
 			(at 0 0 0)
 			(layer "F.SilkS")
+			(hide yes)
 			(effects
 				(font
@@
 		(property "Value" "LOGO"
 			(at 0.75 0 0)
-			(layer "F.SilkS")
+			(layer "B.SilkS")
 			(hide yes)
 			(effects
@@
 					(thickness 0.3)
 				)
+				(justify mirror)
 			)
 		)
@@
 		(tags "Arduino Nano")
 		(property "Reference" "A1"
-			(at 7.62 43.05 180)
+			(at 7.62 43.05 0)
 			(layer "F.SilkS")
 			(hide yes)
@@
 		(layer "Edge.Cuts")
 	)
-	(gr_text "A1"
-		(at 160.3 117.9 180)
+	(gr_text "P+"
+		(at 183.4 58 180)
 		(layer "F.SilkS")
 		(effects
@@
 		)
 	)
-	(gr_text "A2\n"
-		(at 180.7 117.6 180)
+	(gr_text "D+"
+		(at 181.4 58 180)
 		(layer "F.SilkS")
 		(effects
@@
 		)
 	)
-	(gr_text "P+\n"
-		(at 163.8 59.3 0)
-		(layer "B.SilkS")
+	(gr_text "D-"
+		(at 177.4 58 180)
+		(layer "F.SilkS")
 		(effects
 			(font
 				(size 1 1)
-				(thickness 0.15)
+				(thickness 0.1)
 			)
-			(justify left bottom mirror)
+			(justify left bottom)
 		)
 	)
-	(gr_text "D-"
-		(at 177 59.3 0)
-		(layer "B.SilkS")
+	(gr_text "D+"
+		(at 161.2 58.2 180)
+		(layer "F.SilkS")
 		(effects
 			(font
 				(size 1 1)
-				(thickness 0.15)
+				(thickness 0.1)
 			)
-			(justify left bottom mirror)
+			(justify left bottom)
 		)
 	)
-	(gr_text "P-"
-		(at 159.4 59.3 0)
-		(layer "B.SilkS")
+	(gr_text "A1"
+		(at 160.3 117.9 180)
+		(layer "F.SilkS")
 		(effects
 			(font
 				(size 1 1)
-				(thickness 0.15)
+				(thickness 0.1)
 			)
-			(justify left bottom mirror)
+			(justify left bottom)
 		)
 	)
-	(gr_text "P+\n"
-		(at 183.5 59.3 0)
-		(layer "B.SilkS")
+	(gr_text "D-"
+		(at 157.2 58.2 180)
+		(layer "F.SilkS")
 		(effects
 			(font
 				(size 1 1)
-				(thickness 0.15)
+				(thickness 0.1)
 			)
-			(justify left bottom mirror)
+			(justify left bottom)
 		)
 	)
-	(gr_text "D+\n"
-		(at 161.5 59.3 0)
-		(layer "B.SilkS")
+	(gr_text "P+"
+		(at 163.2 58.2 180)
+		(layer "F.SilkS")
 		(effects
 			(font
 				(size 1 1)
-				(thickness 0.15)
+				(thickness 0.1)
 			)
-			(justify left bottom mirror)
+			(justify left bottom)
 		)
 	)
-	(gr_text "D-"
-		(at 157.3 59.3 0)
-		(layer "B.SilkS")
+	(gr_text "P-"
+		(at 179.4 58 180)
+		(layer "F.SilkS")
 		(effects
 			(font
 				(size 1 1)
-				(thickness 0.15)
+				(thickness 0.1)
 			)
-			(justify left bottom mirror)
+			(justify left bottom)
 		)
 	)
-	(gr_text "P-"
-		(at 179.1 59.3 0)
-		(layer "B.SilkS")
+	(gr_text "A2\n"
+		(at 180.7 117.6 180)
+		(layer "F.SilkS")
 		(effects
 			(font
 				(size 1 1)
-				(thickness 0.15)
+				(thickness 0.1)
 			)
-			(justify left bottom mirror)
+			(justify left bottom)
 		)
 	)
-	(gr_text "D+\n"
-		(at 181.2 59.3 0)
-		(layer "B.SilkS")
+	(gr_text "P-"
+		(at 159.2 58.2 180)
+		(layer "F.SilkS")
 		(effects
 			(font
 				(size 1 1)
-				(thickness 0.15)
+				(thickness 0.1)
 			)
-			(justify left bottom mirror)
+			(justify left bottom)
 		)
 	)
@@
 		(end 151.89 102.89)
 		(width 0.4)
-		(layer "F.Cu")
+		(layer "B.Cu")
 		(net 3)
 	)
@@
 		(end 162.5 92.28)
 		(width 0.4)
-		(layer "F.Cu")
+		(layer "B.Cu")
 		(net 3)
 	)
@@
 		(end 160.5 67.6)
 		(width 0.4)
-		(layer "F.Cu")
+		(layer "B.Cu")
 		(net 6)
 	)
@@
 		(end 151.89 85.11)
 		(width 0.4)
-		(layer "F.Cu")
+		(layer "B.Cu")
 		(net 6)
 	)
@@
 		(end 160.9 65.2)
 		(width 0.4)
-		(layer "F.Cu")
+		(layer "B.Cu")
 		(net 23)
 	)
@@
 		(end 156.5 67.6)
 		(width 0.4)
-		(layer "F.Cu")
+		(layer "B.Cu")
 		(net 23)
 	)
@@
 		(end 174.1 65.2)
 		(width 0.4)
-		(layer "F.Cu")
+		(layer "B.Cu")
 		(net 23)
 	)
@@
 		(end 176.5 67.6)
 		(width 0.4)
-		(layer "F.Cu")
+		(layer "B.Cu")
 		(net 23)
 	)
@@
 		(end 176.5 67.6)
 		(width 0.4)
-		(layer "F.Cu")
+		(layer "B.Cu")
 		(net 23)
 	)
@@
 		(end 176.5 78.08)
 		(width 0.4)
-		(layer "F.Cu")
+		(layer "B.Cu")
 		(net 23)
 	)
@@
 		(end 172 82.58)
 		(width 0.4)
-		(layer "F.Cu")
+		(layer "B.Cu")
 		(net 23)
 	)
@@
 		(end 151.89 82.57)
 		(width 0.4)
-		(layer "F.Cu")
+		(layer "B.Cu")
 		(net 23)
 	)
@@
 		(end 156.5 77.96)
 		(width 0.4)
-		(layer "F.Cu")
+		(layer "B.Cu")
 		(net 23)
 	)
@@
 		(end 172 102.9)
 		(width 0.4)
-		(layer "F.Cu")
+		(layer "B.Cu")
 		(net 45)
 	)
@@
 		(end 182.5 92.4)
 		(width 0.4)
-		(layer "F.Cu")
+		(layer "B.Cu")
 		(net 45)
 	)
@@
 		(end 172 85.12)
 		(width 0.4)
-		(layer "F.Cu")
+		(layer "B.Cu")
 		(net 57)
 	)
@@
 		(end 180.5 76.62)
 		(width 0.4)
-		(layer "F.Cu")
+		(layer "B.Cu")
 		(net 57)
 	)
@@
 		(net 23)
 		(net_name "DIR- 1")
-		(layer "F.Cu")
+		(layer "B.Cu")
 		(hatch edge 0.5)
 		(connect_pads
